File: hum_hw.kicad_pcb (KiCad board)
At the start: 4 copper layers, 50.8 x 50.8 mm, 31 parts, among them J1 Conn_01x02_Pin, J2 Conn_01x03, J3 Conn_ARM_JTAG_SWD_10, J4 Conn_01x02_Pin, SW1 SW_SPST, U1 24FC512-I/ST, U2 STM32U031K8U6, U4 LIS2DTW12TR, Y1 32.768kHZ

Commit message: brd layout
Parts:
- removed R4: 4.7k, Resistor_SMD:R_0805_2012Metric
- added R9: 1k, Resistor_SMD:R_0805_2012Metric, F.Cu at (240.7, 123.8)
- C4, C5, C6, C7, C8, C9: moved to B.Cu
- moved U1 151.8 mm to (252.7, 118.1), turned to -90 degrees
- moved SW1 151.3 mm to (237.7, 112.0), turned to 90 degrees
- moved J3 148.5 mm to (249.0, 126.4)
- moved J2 144.4 mm to (237.5, 127.0), turned to 90 degrees
- moved R5 141.6 mm to (248.9, 120.0), turned to 180 degrees
- moved R6 140.7 mm to (248.9, 118.1), turned to 180 degrees
- moved R7 140.0 mm to (248.9, 116.2), turned to 180 degrees
- moved C10 139.6 mm to (255.3, 118.1), turned to -90 degrees
- moved U2 132.7 mm to (242.6, 118.7), turned to -90 degrees
- moved C4 132.6 mm to (244.3, 116.9), turned to -90 degrees
- moved C6 131.0 mm to (242.6, 120.2), turned to 90 degrees
- moved R1 130.8 mm to (237.2, 117.2), turned to 90 degrees
- moved C3 130.0 mm to (242.6, 109.7), turned to 90 degrees
- moved Y1 129.7 mm to (243.9, 112.5)
- moved C1 129.2 mm to (240.8, 112.3), turned to 90 degrees
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Connections:
- J2 pad 2: /PA10_RX1 -> /_PA10_RX1

Commit message: brd layout complete
Parts:
- removed J4: Conn_01x02_Pin, Connector_PinHeader_2.54mm:PinHeader_1x02_P2.54mm_Vertical
- BT1, J3: moved to B.Cu
- C13: renamed from C1; moved to B.Cu
- C6: renamed from C10; moved to B.Cu
- R6: renamed from R9; moved to B.Cu
- SW1: footprint CandK3:SWITCH_4.20X2.80_revB -> Button_Switch_SMD:SW_SPST_PTS645Sx43SMTR92
- moved R1 156.0 mm to (93.3, 105.0)
- moved R3 156.0 mm to (93.3, 106.9)
- moved R4 156.0 mm to (93.3, 108.8)
- moved U1 155.8 mm to (97.2, 110.1)
- moved C6 155.7 mm to (99.6, 114.9)
- moved C8 155.5 mm to (90.9, 114.9)
- moved C1 155.1 mm to (87.5, 108.0)
- moved Y1 155.1 mm to (88.8, 110.7)
- moved D2 155.1 mm to (82.3, 115.4), turned to -90 degrees
- moved C2 154.9 mm to (90.2, 108.0)
- moved R5 154.9 mm to (82.3, 119.1), turned to -90 degrees
- moved C10 154.7 mm to (86.1, 114.9)
- moved C9 154.7 mm to (87.9, 114.9)
- moved C12 154.4 mm to (86.4, 119.4)
- moved C11 154.4 mm to (88.1, 119.4)
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- renumbered C3 to C1, C8 to C10, C6 to C11, C7 to C12, C12 to C2, C2 to C3, C13 to C4, C14 to C5, C4 to C7, C5 to C8, D2 to D1, D1 to D2, R7 to R1, R8 to R2, R6 to R3, R5 to R4, R1 to R5, U4 to U3
Connections:
- net /B+ renamed Net-(BT1-+)
Routing:
- net VCC: track 0.00 -> 42.2 mm, vias 0 -> 12
- net Net-(BT1-+): track 0.00 -> 35.9 mm, vias 0 -> 14
- net /~{PF2_RST}: track 0.00 -> 27.4 mm, vias 0 -> 1
- net /PA1_SWT: track 0.00 -> 22.6 mm
- net /PB6_SCL: track 0.00 -> 20.9 mm, vias 0 -> 2
- net /PA2_AINT2: track 0.00 -> 20.0 mm, vias 0 -> 2
- net /PB7_SDA: track 0.00 -> 18.7 mm, vias 0 -> 2
- net GND: track 0.00 -> 18.5 mm, vias 0 -> 36
- net /PA13_SWDIO: track 0.00 -> 16.7 mm, vias 0 -> 1
- net /PA0_AINT1: track 0.00 -> 16.4 mm, vias 0 -> 2
- net Net-(U2-PF3): track 0.00 -> 14.8 mm
- net /PA14_SWCLK: track 0.00 -> 14.8 mm, vias 0 -> 1
- net /PA8_LED: track 0.00 -> 7.53 mm
- net Net-(U2-PC15): track 0.00 -> 7.27 mm
- net /PA9_TX1: track 0.00 -> 6.94 mm
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- added copper zone on B.Cu, net GND
- added copper zone on F.Cu, net GND
- added copper zone on In1.Cu, net GND
- added copper zone on In2.Cu, net GND
- added copper zone on In2.Cu, net VCC
Other:
- board size 50.8 x 50.8 mm -> 25.4 x 43.2 mm
- board text added: "3V ONLY"
- board text added: "CR2032"
- board text added: "GND"
- board text added: "HUM_HW V1.0.0 TACTICAL_SNACKS 20261014"
- board text added: "ISNS"
- board text added: "RX"
- board text added: "TX"
