File: hum_hw.kicad_sch (KiCad schematic)
At the start: 30 parts, among them J1 Conn_01x02_Pin, J2 Conn_01x03, J3 Conn_ARM_JTAG_SWD_10, J4 Conn_01x02_Pin, SW1 SW_SPST, U1 24FC512-I/ST, U2 STM32U031K8U6, U4 LIS2DTW12TR, Y1 32.768kHZ

Commit message: brd layout
Parts:
- added R9: 1k, Resistor_SMD:R_0805_2012Metric, symbol Device:R_Small
Connections:
- net PA10_RX1: now also R9.2; no longer J2.2 (Pin_2)
- new net _PA10_RX1: J2.2 (Pin_2), R9.1
Changed lines of the file:
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@@
+	(wire
+		(pts
+			(xy 242.57 148.59) (xy 255.27 148.59)
+		)
+		(stroke
+			(width 0)
+			(type default)
+		)
+	)
 	(wire
 		(pts
@@
 	)
 	(label "PA10_RX1"
-		(at 255.27 148.59 180)
+		(at 237.49 148.59 180)
 		(effects
 			(font
@@
 			)
 			(justify left bottom)
+		)
+	)
+	(label "_PA10_RX1"
+		(at 255.27 148.59 180)
+		(effects
+			(font
+				(size 1.27 1.27)
+			)
+			(justify right bottom)
 		)
 	)
@@
 					(unit 1)
 				)
+			)
+		)
+	)
+	(symbol
+		(lib_id "Device:R_Small")
+		(at 240.03 148.59 270)
+		(mirror x)
+		(unit 1)
+		(body_style 1)
+		(exclude_from_sim no)
+		(in_bom yes)
+		(on_board yes)
+		(in_pos_files yes)
+		(dnp no)
+		(fields_autoplaced yes)
+		(property "Reference" "R9"
+			(at 240.03 143.51 90)
+			(show_name no)
+			(do_not_autoplace no)
+			(effects
+				(font
+					(size 1.016 1.016)
+				)
+			)
+		)
+		(property "Value" "1k"
+			(at 240.03 146.05 90)
+			(show_name no)
+			(do_not_autoplace no)
+			(effects
+				(font
+					(size 1.27 1.27)
+				)
+			)
+		)
+		(property "Footprint" "Resistor_SMD:R_0805_2012Metric"
+			(at 240.03 148.59 0)
+			(hide yes)
+			(show_name no)
+			(do_not_autoplace no)
+			(effects
+				(font
+					(size 1.27 1.27)
+				)
+			)
+		)
+		(property "Datasheet" ""
+			(at 240.03 148.59 0)
+			(hide yes)
+			(show_name no)
+			(do_not_autoplace no)
+			(effects
+				(font
+					(size 1.27 1.27)
+				)
+			)
+		)
+		(property "Description" "Resistor, small symbol"
+			(at 240.03 148.59 0)
+			(hide yes)
+			(show_name no)
+			(do_not_autoplace no)
+			(effects
+				(font
+					(size 1.27 1.27)
+				)
+			)
+		)
+		(property "MFR" ""
+			(at 240.03 148.59 0)
+			(hide yes)
+			(show_name no)
+			(do_not_autoplace no)
+			(effects
+				(font
+					(size 1.27 1.27)
+				)
+			)
+		)
+		(property "MFR_PN" ""
+			(at 240.03 148.59 0)
+			(hide yes)
+			(show_name no)
+			(do_not_autoplace no)
+			(effects
+				(font
+					(size 1.27 1.27)
+				)
+			)
+		)
+		(property "VENDOR" ""
+			(at 240.03 148.59 0)
+			(hide yes)
+			(show_name no)
+			(do_not_autoplace no)
+			(effects
+				(font
+					(size 1.27 1.27)
+				)
+			)
+		)
+		(property "VENDOR_PN" ""
+			(at 240.03 148.59 0)
+			(hide yes)
+			(show_name no)
+			(do_not_autoplace no)
+			(effects
+				(font
+					(size 1.27 1.27)
+				)
+			)
+		)
+		(property "VENDOR_DESC" ""
+			(at 240.03 148.59 0)
+			(hide yes)
+			(show_name no)
+			(do_not_autoplace no)
+			(effects
+				(font
+					(size 1.27 1.27)
+				)
+			)
+		)
+		(property "ALT" ""
+			(at 240.03 148.59 0)
+			(hide yes)
+			(show_name no)
+			(do_not_autoplace no)
+			(effects
+				(font
+					(size 1.27 1.27)
+				)
+			)
+		)
+		(property "Purpose" ""
+			(at 240.03 148.59 0)
+			(hide yes)
+			(show_name no)
+			(do_not_autoplace no)
+			(effects
+				(font
+					(size 1.27 1.27)
+				)
+			)
+		)
+		(pin "2"
+		)
+		(pin "1"
+		)
+		(instances
+			(project "hum_hw"
+				(path "/3ce56f88-c583-47ce-a098-cbd585c70caf"
+					(reference "R9")
+					(unit 1)
+				)

Commit message: brd layout complete
Parts:
- removed J4: Conn_01x02_Pin, Connector_PinHeader_2.54mm:PinHeader_1x02_P2.54mm_Vertical, symbol Connector:Conn_01x02_Pin
- R2: renamed from R8; Purpose (none) -> CURRENT_SENSE
- SW1: footprint CandK3:SWITCH_4.20X2.80_revB -> Button_Switch_SMD:SW_SPST_PTS645Sx43SMTR92
- renumbered C3 to C1, C8 to C10, C6 to C11, C7 to C12, C1 to C13, C12 to C2, C2 to C3, C13 to C4, C14 to C5, C10 to C6, C4 to C7, C5 to C8, D2 to D1, D1 to D2, R7 to R1, R6 to R3, R5 to R4, R1 to R5, R9 to R6, U4 to U3
Connections:
- net B+: no longer names the net of BT1.1 (+), R2.1
Other:
- moved on the sheet: R2

Commit message: stp, renders, datasheets
Parts:
- J3: MFR (none) -> GCT; MFR_PN (none) -> BD125-10-A-0305-0580-L-B; VENDOR (none) -> Digi-Key; VENDOR_DESC (none) -> HEADER DUAL 1.27MM VERT SMT 10POS; VENDOR_PN (none) -> 2073-BD125-10-A-0305-0580-L-BCT-ND
Changed lines of the file:
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@@
+			)
+		)
+		(property "MFR" "GCT"
+			(at 123.19 165.1 0)
+			(hide yes)
+			(show_name no)
+			(do_not_autoplace no)
+			(effects
+				(font
+					(size 1.27 1.27)
+				)
+			)
+		)
+		(property "MFR_PN" "BD125-10-A-0305-0580-L-B"
+			(at 123.19 165.1 0)
+			(hide yes)
+			(show_name no)
+			(do_not_autoplace no)
+			(effects
+				(font
+					(size 1.27 1.27)
+				)
+			)
+		)
+		(property "VENDOR" "Digi-Key"
+			(at 123.19 165.1 0)
+			(hide yes)
+			(show_name no)
+			(do_not_autoplace no)
+			(effects
+				(font
+					(size 1.27 1.27)
+				)
+			)
+		)
+		(property "VENDOR_DESC" "HEADER DUAL 1.27MM VERT SMT 10POS"
+			(at 123.19 165.1 0)
+			(hide yes)
+			(show_name no)
+			(do_not_autoplace no)
+			(effects
+				(font
+					(size 1.27 1.27)
+				)
+			)
+		)
+		(property "VENDOR_PN" "2073-BD125-10-A-0305-0580-L-BCT-ND"
+			(at 123.19 165.1 0)
+			(hide yes)
+			(show_name no)
+			(do_not_autoplace no)
+			(effects
+				(font
+					(size 1.27 1.27)
+				)
 			)
 		)

Commit message: pics, areas of improvement
Other:
- note added: "REVISION INFO V1.0.0 - INITIAL DESIGN AREAS OF IMPROVEMENT - CONSOLIDATE 0603/0805 - PROG HEADER PLACEMENT IS TERRIBLE, HANGS OVER BOARD EDGE, INTERFERES WITH CAP"
- note removed: "REVISION INFO V1.0 - INITIAL DESIGN"
Changed lines of the file:
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@@
 		)
 	)
-	(text "REVISION INFO\n\nV1.0 - INITIAL DESIGN"
+	(text "REVISION INFO\n\nV1.0.0 - INITIAL DESIGN\n\nAREAS OF IMPROVEMENT\n- CONSOLIDATE 0603/0805\n- PROG HEADER PLACEMENT IS TERRIBLE, HANGS OVER BOARD EDGE, INTERFERES WITH CAP"
 		(exclude_from_sim no)
 		(at 16.51 194.31 0)

Commit message: title block, pdf
Other:
- company: (none) -> TACTICAL SNACKS
- title: TITLE -> HUM_HW
Changed lines of the file:
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@@
 	(paper "A4")
 	(title_block
-		(title "TITLE")
+		(title "HUM_HW")
+		(date "2026-10-14")
+		(rev "1.0.0")
+		(company "TACTICAL SNACKS")
 	)
 	(text "VDDA"
